File: PCB/PCB Card/PCB Card.kicad_sch (KiCad schematic)
At the start: 5 parts, among them U1 NT3H2111W0FHKH

Commit message: antenna and placement
Parts:
- AE1: footprint (none) -> KiCad_Package:NFC_30x30_N5_Custom_YOLO_Mode
- C1: footprint (none) -> Capacitor_SMD:C_0201_0603Metric
- D1: footprint (none) -> LED_SMD:LED_0805_2012Metric
- R1: footprint (none) -> Resistor_SMD:R_0201_0603Metric
- U1: footprint kicad_why:XQFN-8_L1.6-W1.6-P0.50-BL_NT3H2111W0FHKH -> Project Resources:XQFN-8_L1.6-W1.6-P0.50-BL_NT3H2111W0FHKH
Changed lines of the file:
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@@
 			)
 		)
-		(property "Footprint" ""
+		(property "Footprint" "Resistor_SMD:R_0201_0603Metric"
 			(at 135.89 107.188 90)
 			(hide yes)
@@
 			)
 		)
-		(property "Footprint" ""
+		(property "Footprint" "LED_SMD:LED_0805_2012Metric"
 			(at 110.49 105.41 0)
 			(hide yes)
@@
 			)
 		)
-		(property "Footprint" ""
+		(property "Footprint" "Capacitor_SMD:C_0201_0603Metric"
 			(at 125.73 90.4748 0)
 			(hide yes)
@@
 			)
 		)
-		(property "Footprint" ""
+		(property "Footprint" "KiCad_Package:NFC_30x30_N5_Custom_YOLO_Mode"
 			(at 121.92 45.72 0)
 			(hide yes)
@@
 			)
 		)
-		(property "Footprint" "kicad_why:XQFN-8_L1.6-W1.6-P0.50-BL_NT3H2111W0FHKH"
+		(property "Footprint" "Project Resources:XQFN-8_L1.6-W1.6-P0.50-BL_NT3H2111W0FHKH"
 			(at 121.92 83.82 0)
 			(hide yes)
